Commit message: Update joint limits + scaling factors

File: so_arm100_description/urdf/so_arm100.urdf (robot description, URDF)
Before this commit: robot so_arm100, 7 links, 6 joints
Joints:
- joint elbow_joint: limit (none) -> lower=-1.75 upper=1.57 effort=1 velocity=1; type continuous -> revolute
- joint jaw_joint: limit (none) -> lower=-0.22 upper=2.0 effort=1 velocity=1; type continuous -> revolute
- joint shoulder_lift_joint: limit (none) -> lower=-1.75 upper=1.75 effort=1 velocity=1; type continuous -> revolute
- joint shoulder_pan_joint: axis 0 1 0 -> 0 -1 0; limit (none) -> lower=-2.0 upper=2.0 effort=1 velocity=1; type continuous -> revolute
- joint wrist_pitch_joint: limit (none) -> lower=-3.5 upper=0.2 effort=1 velocity=1; type continuous -> revolute
- joint wrist_roll_joint: limit (none) -> lower=-1.0 upper=4.0 effort=1 velocity=1; type continuous -> revolute
