Commit message: removes submodule and adds meshes

File: so_arm100_description/urdf/so_arm100_macro.xacro (robot description, xacro)
@@ -27,21 +27,21 @@
         <geometry>
           <mesh
-            filename="package://so_arm100_description/SO100/assets/Base.stl"
-          />
-        </geometry>
-        <material name="3d_printed" />
-      </visual>
-      <visual>
-        <geometry>
-          <mesh
-            filename="package://so_arm100_description/SO100/assets/Base_Motor.stl"
-          />
-        </geometry>
-        <material name="sts3215" />
-      </visual>
-      <collision>
-        <geometry>
-          <mesh
-            filename="package://so_arm100_description/SO100/assets/Base.stl"
+            filename="package://so_arm100_description/meshes/Base.stl"
+          />
+        </geometry>
+        <material name="3d_printed" />
+      </visual>
+      <visual>
+        <geometry>
+          <mesh
+            filename="package://so_arm100_description/meshes/Base_Motor.stl"
+          />
+        </geometry>
+        <material name="sts3215" />
+      </visual>
+      <collision>
+        <geometry>
+          <mesh
+            filename="package://so_arm100_description/meshes/Base.stl"
           />
         </geometry>
@@ -65,21 +65,21 @@
         <geometry>
           <mesh
-            filename="package://so_arm100_description/SO100/assets/Rotation_Pitch.stl"
-          />
-        </geometry>
-        <material name="3d_printed" />
-      </visual>
-      <visual>
-        <geometry>
-          <mesh
-            filename="package://so_arm100_description/SO100/assets/Rotation_Pitch_Motor.stl"
-          />
-        </geometry>
-        <material name="sts3215" />
-      </visual>
-      <collision>
-        <geometry>
-          <mesh
-            filename="package://so_arm100_description/SO100/assets/Rotation_Pitch.stl"
+            filename="package://so_arm100_description/meshes/Rotation_Pitch.stl"
+          />
+        </geometry>
+        <material name="3d_printed" />
+      </visual>
+      <visual>
+        <geometry>
+          <mesh
+            filename="package://so_arm100_description/meshes/Rotation_Pitch_Motor.stl"
+          />
+        </geometry>
+        <material name="sts3215" />
+      </visual>
+      <collision>
+        <geometry>
+          <mesh
+            filename="package://so_arm100_description/meshes/Rotation_Pitch.stl"
           />
         </geometry>
@@ -103,21 +103,21 @@
         <geometry>
           <mesh
-            filename="package://so_arm100_description/SO100/assets/Upper_Arm.stl"
-          />
-        </geometry>
-        <material name="3d_printed" />
-      </visual>
-      <visual>
-        <geometry>
-          <mesh
-            filename="package://so_arm100_description/SO100/assets/Upper_Arm_Motor.stl"
-          />
-        </geometry>
-        <material name="sts3215" />
-      </visual>
-      <collision>
-        <geometry>
-          <mesh
-            filename="package://so_arm100_description/SO100/assets/Upper_Arm.stl"
+            filename="package://so_arm100_description/meshes/Upper_Arm.stl"
+          />
+        </geometry>
+        <material name="3d_printed" />
+      </visual>
+      <visual>
+        <geometry>
+          <mesh
+            filename="package://so_arm100_description/meshes/Upper_Arm_Motor.stl"
+          />
+        </geometry>
+        <material name="sts3215" />
+      </visual>
+      <collision>
+        <geometry>
+          <mesh
+            filename="package://so_arm100_description/meshes/Upper_Arm.stl"
           />
         </geometry>
@@ -141,21 +141,21 @@
         <geometry>
           <mesh
-            filename="package://so_arm100_description/SO100/assets/Lower_Arm.stl"
-          />
-        </geometry>
-        <material name="3d_printed" />
-      </visual>
-      <visual>
-        <geometry>
-          <mesh
-            filename="package://so_arm100_description/SO100/assets/Lower_Arm_Motor.stl"
-          />
-        </geometry>
-        <material name="sts3215" />
-      </visual>
-      <collision>
-        <geometry>
-          <mesh
-            filename="package://so_arm100_description/SO100/assets/Lower_Arm.stl"
+            filename="package://so_arm100_description/meshes/Lower_Arm.stl"
+          />
+        </geometry>
+        <material name="3d_printed" />
+      </visual>
+      <visual>
+        <geometry>
+          <mesh
+            filename="package://so_arm100_description/meshes/Lower_Arm_Motor.stl"
+          />
+        </geometry>
+        <material name="sts3215" />
+      </visual>
+      <collision>
+        <geometry>
+          <mesh
+            filename="package://so_arm100_description/meshes/Lower_Arm.stl"
           />
         </geometry>
@@ -179,21 +179,21 @@
         <geometry>
           <mesh
-            filename="package://so_arm100_description/SO100/assets/Wrist_Pitch_Roll.stl"
-          />
-        </geometry>
-        <material name="3d_printed" />
-      </visual>
-      <visual>
-        <geometry>
-          <mesh
-            filename="package://so_arm100_description/SO100/assets/Wrist_Pitch_Roll_Motor.stl"
-          />
-        </geometry>
-        <material name="sts3215" />
-      </visual>
-      <collision>
-        <geometry>
-          <mesh
-            filename="package://so_arm100_description/SO100/assets/Wrist_Pitch_Roll.stl"
+            filename="package://so_arm100_description/meshes/Wrist_Pitch_Roll.stl"
+          />
+        </geometry>
+        <material name="3d_printed" />
+      </visual>
+      <visual>
+        <geometry>
+          <mesh
+            filename="package://so_arm100_description/meshes/Wrist_Pitch_Roll_Motor.stl"
+          />
+        </geometry>
+        <material name="sts3215" />
+      </visual>
+      <collision>
+        <geometry>
+          <mesh
+            filename="package://so_arm100_description/meshes/Wrist_Pitch_Roll.stl"
           />
         </geometry>
@@ -217,13 +217,13 @@
         <geometry>
           <mesh
-            filename="package://so_arm100_description/SO100/assets/Fixed_Jaw.stl"
-          />
-        </geometry>
-        <material name="3d_printed" />
-      </visual>
-      <visual>
-        <geometry>
-          <mesh
-            filename="package://so_arm100_description/SO100/assets/Fixed_Jaw_Motor.stl"
+            filename="package://so_arm100_description/meshes/Fixed_Jaw.stl"
+          />
+        </geometry>
+        <material name="3d_printed" />
+      </visual>
+      <visual>
+        <geometry>
+          <mesh
+            filename="package://so_arm100_description/meshes/Fixed_Jaw_Motor.stl"
           />
         </geometry>
@@ -248,5 +248,5 @@
         <geometry>
           <mesh
-            filename="package://so_arm100_description/SO100/assets/Moving_Jaw.stl"
+            filename="package://so_arm100_description/meshes/Moving_Jaw.stl"
           />
         </geometry>

File: so_arm101_description/urdf/so_arm101.urdf.xacro (robot description, xacro)
@@ -12,5 +12,5 @@
   <xacro:arg name="usb_port" default="/dev/LeRobotFollower" />
   <xacro:arg name="prefix" default="" />
-  <xacro:arg name="color" default="1.0 0.82 0.12 1.0" />
+  <xacro:arg name="color" default="0.2 0.7 0.85 1.0" />
   <!-- Robot description -->
   <xacro:include filename="$(arg urdf_file)" />

File: so_arm101_description/urdf/so_arm101_macro.xacro (robot description, xacro)
@@ -1,5 +1,5 @@
 <?xml version="1.0" encoding="utf-8" ?>
 <robot xmlns:xacro="http://ros.org/wiki/xacro">
-  <xacro:macro name="so_arm101" params="prefix color:='1.0 0.82 0.12 1.0'">
+  <xacro:macro name="so_arm101" params="prefix color:='0.2 0.7 0.85 1.0'">
     <!-- Materials -->
     <material name="3d_printed">
@@ -20,5 +20,5 @@
         <origin xyz="-0.00636471 -9.94414e-05 -0.0024" rpy="1.5708 -1.67685e-15 1.5708"/>
         <geometry>
-          <mesh filename="package://so_arm100_description/SO101/assets/base_motor_holder_so101_v1.stl"/>
+          <mesh filename="package://so_arm101_description/meshes/base_motor_holder_so101_v1.stl"/>
         </geometry>
         <material name="3d_printed"/>
@@ -27,5 +27,5 @@
         <origin xyz="-0.00636471 -9.94414e-05 -0.0024" rpy="1.5708 -1.67685e-15 1.5708"/>
         <geometry>
-          <mesh filename="package://so_arm100_description/SO101/assets/base_motor_holder_so101_v1.stl"/>
+          <mesh filename="package://so_arm101_description/meshes/base_motor_holder_so101_v1.stl"/>
         </geometry>
       </collision>
@@ -34,5 +34,5 @@
         <origin xyz="-0.00636471 -8.97657e-09 -0.0024" rpy="1.5708 -2.78073e-29 1.5708"/>
         <geometry>
-          <mesh filename="package://so_arm100_description/SO101/assets/base_so101_v2.stl"/>
+          <mesh filename="package://so_arm101_description/meshes/base_so101_v2.stl"/>
         </geometry>
         <material name="3d_printed"/>
@@ -41,5 +41,5 @@
         <origin xyz="-0.00636471 -8.97657e-09 -0.0024" rpy="1.5708 -2.78073e-29 1.5708"/>
         <geometry>
-          <mesh filename="package://so_arm100_description/SO101/assets/base_so101_v2.stl"/>
+          <mesh filename="package://so_arm101_description/meshes/base_so101_v2.stl"/>
         </geometry>
       </collision>
@@ -48,12 +48,12 @@
         <origin xyz="0.0263353 -8.97657e-09 0.0437" rpy="-8.21148e-16 7.84513e-18 1.249e-15"/>
         <geometry>
-          <mesh filename="package://so_arm100_description/SO101/assets/sts3215_03a_v1.stl"/>
-        </geometry>
-        <material name="sts3215"/>
+          <mesh filename="package://so_arm101_description/meshes/sts3215_03a_v1.stl"/>
+        </geometry>
+        <material name="3d_printed"/>
       </visual>
       <collision>
         <origin xyz="0.0263353 -8.97657e-09 0.0437" rpy="-8.21148e-16 7.84513e-18 1.249e-15"/>
         <geometry>
-          <mesh filename="package://so_arm100_description/SO101/assets/sts3215_03a_v1.stl"/>
+          <mesh filename="package://so_arm101_description/meshes/sts3215_03a_v1.stl"/>
         </geometry>
       </collision>
@@ -62,5 +62,5 @@
         <origin xyz="-0.0309827 -0.000199441 0.0474" rpy="1.5708 -1.35493e-14 1.5708"/>
         <geometry>
-          <mesh filename="package://so_arm100_description/SO101/assets/waveshare_mounting_plate_so101_v2.stl"/>
+          <mesh filename="package://so_arm101_description/meshes/waveshare_mounting_plate_so101_v2.stl"/>
         </geometry>
         <material name="3d_printed"/>
@@ -69,5 +69,5 @@
         <origin xyz="-0.0309827 -0.000199441 0.0474" rpy="1.5708 -1.35493e-14 1.5708"/>
         <geometry>
-          <mesh filename="package://so_arm100_description/SO101/assets/waveshare_mounting_plate_so101_v2.stl"/>
+          <mesh filename="package://so_arm101_description/meshes/waveshare_mounting_plate_so101_v2.stl"/>
         </geometry>
       </collision>
@@ -84,12 +84,12 @@
         <origin xyz="-0.0303992 0.000422241 -0.0417" rpy="1.5708 1.5708 0"/>
         <geometry>
-          <mesh filename="package://so_arm100_description/SO101/assets/sts3215_03a_v1.stl"/>
-        </geometry>
-        <material name="sts3215"/>
+          <mesh filename="package://so_arm101_description/meshes/sts3215_03a_v1.stl"/>
+        </geometry>
+        <material name="3d_printed"/>
       </visual>
       <collision>
         <origin xyz="-0.0303992 0.000422241 -0.0417" rpy="1.5708 1.5708 0"/>
         <geometry>
-          <mesh filename="package://so_arm100_description/SO101/assets/sts3215_03a_v1.stl"/>
+          <mesh filename="package://so_arm101_description/meshes/sts3215_03a_v1.stl"/>
         </geometry>
       </collision>
@@ -98,5 +98,5 @@
         <origin xyz="-0.0675992 -0.000177759 0.0158499" rpy="1.5708 -1.5708 0"/>
         <geometry>
-          <mesh filename="package://so_arm100_description/SO101/assets/motor_holder_so101_base_v1.stl"/>
+          <mesh filename="package://so_arm101_description/meshes/motor_holder_so101_base_v1.stl"/>
         </geometry>
         <material name="3d_printed"/>
@@ -105,5 +105,5 @@
         <origin xyz="-0.0675992 -0.000177759 0.0158499" rpy="1.5708 -1.5708 0"/>
         <geometry>
-          <mesh filename="package://so_arm100_description/SO101/assets/motor_holder_so101_base_v1.stl"/>
+          <mesh filename="package://so_arm101_description/meshes/motor_holder_so101_base_v1.stl"/>
         </geometry>
       </collision>
@@ -112,5 +112,5 @@
         <origin xyz="0.0122008 2.22413e-05 0.0464" rpy="-1.5708 2.35221e-33 0"/>
         <geometry>
-          <mesh filename="package://so_arm100_description/SO101/assets/rotation_pitch_so101_v1.stl"/>
+          <mesh filename="package://so_arm101_description/meshes/rotation_pitch_so101_v1.stl"/>
         </geometry>
         <material name="3d_printed"/>
@@ -119,5 +119,5 @@
         <origin xyz="0.0122008 2.22413e-05 0.0464" rpy="-1.5708 2.35221e-33 0"/>
         <geometry>
-          <mesh filename="package://so_arm100_description/SO101/assets/rotation_pitch_so101_v1.stl"/>
+          <mesh filename="package://so_arm101_description/meshes/rotation_pitch_so101_v1.stl"/>
         </geometry>
       </collision>
@@ -134,12 +134,12 @@
         <origin xyz="-0.11257 -0.0155 0.0187" rpy="-3.14159 -5.27356e-16 -1.5708"/>
         <geometry>
-          <mesh filename="package://so_arm100_description/SO101/assets/sts3215_03a_v1.stl"/>
-        </geometry>
-        <material name="sts3215"/>
+          <mesh filename="package://so_arm101_description/meshes/sts3215_03a_v1.stl"/>
+        </geometry>
+        <material name="3d_printed"/>
       </visual>
       <collision>
         <origin xyz="-0.11257 -0.0155 0.0187" rpy="-3.14159 -5.27356e-16 -1.5708"/>
         <geometry>
-          <mesh filename="package://so_arm100_description/SO101/assets/sts3215_03a_v1.stl"/>
+          <mesh filename="package://so_arm101_description/meshes/sts3215_03a_v1.stl"/>
         </geometry>
       </collision>
@@ -148,5 +148,5 @@
         <origin xyz="-0.065085 0.012 0.0182" rpy="3.14159 -0 -1.30911e-30"/>
         <geometry>
-          <mesh filename="package://so_arm100_description/SO101/assets/upper_arm_so101_v1.stl"/>
+          <mesh filename="package://so_arm101_description/meshes/upper_arm_so101_v1.stl"/>
         </geometry>
         <material name="3d_printed"/>
@@ -155,5 +155,5 @@
         <origin xyz="-0.065085 0.012 0.0182" rpy="3.14159 -0 -1.30911e-30"/>
         <geometry>
-          <mesh filename="package://so_arm100_description/SO101/assets/upper_arm_so101_v1.stl"/>
+          <mesh filename="package://so_arm101_description/meshes/upper_arm_so101_v1.stl"/>
         </geometry>
       </collision>
@@ -170,5 +170,5 @@
         <origin xyz="-0.0648499 -0.032 0.0182" rpy="3.14159 -0 6.67202e-31"/>
         <geometry>
-          <mesh filename="package://so_arm100_description/SO101/assets/under_arm_so101_v1.stl"/>
+          <mesh filename="package://so_arm101_description/meshes/under_arm_so101_v1.stl"/>
         </geometry>
         <material name="3d_printed"/>
@@ -177,5 +177,5 @@
         <origin xyz="-0.0648499 -0.032 0.0182" rpy="3.14159 -0 6.67202e-31"/>
         <geometry>
-          <mesh filename="package://so_arm100_description/SO101/assets/under_arm_so101_v1.stl"/>
+          <mesh filename="package://so_arm101_description/meshes/under_arm_so101_v1.stl"/>
         </geometry>
       </collision>
@@ -184,5 +184,5 @@
         <origin xyz="-0.0648499 -0.032 0.018" rpy="-3.14159 -2.55351e-15 -1.83387e-30"/>
         <geometry>
-          <mesh filename="package://so_arm100_description/SO101/assets/motor_holder_so101_wrist_v1.stl"/>
+          <mesh filename="package://so_arm101_description/meshes/motor_holder_so101_wrist_v1.stl"/>
         </geometry>
         <material name="3d_printed"/>
@@ -191,5 +191,5 @@
         <origin xyz="-0.0648499 -0.032 0.018" rpy="-3.14159 -2.55351e-15 -1.83387e-30"/>
         <geometry>
-          <mesh filename="package://so_arm100_description/SO101/assets/motor_holder_so101_wrist_v1.stl"/>
+          <mesh filename="package://so_arm101_description/meshes/motor_holder_so101_wrist_v1.stl"/>
         </geometry>
       </collision>
@@ -198,12 +198,12 @@
         <origin xyz="-0.1224 0.0052 0.0187" rpy="-3.14159 -7.88861e-31 -3.14159"/>
         <geometry>
-          <mesh filename="package://so_arm100_description/SO101/assets/sts3215_03a_v1.stl"/>
-        </geometry>
-        <material name="sts3215"/>
+          <mesh filename="package://so_arm101_description/meshes/sts3215_03a_v1.stl"/>
+        </geometry>
+        <material name="3d_printed"/>
       </visual>
       <collision>
         <origin xyz="-0.1224 0.0052 0.0187" rpy="-3.14159 -7.88861e-31 -3.14159"/>
         <geometry>
-          <mesh filename="package://so_arm100_description/SO101/assets/sts3215_03a_v1.stl"/>
+          <mesh filename="package://so_arm101_description/meshes/sts3215_03a_v1.stl"/>
         </geometry>
       </collision>
@@ -220,12 +220,12 @@
         <origin xyz="8.32667e-17 -0.0424 0.0306" rpy="1.5708 1.5708 0"/>
         <geometry>
-          <mesh filename="package://so_arm100_description/SO101/assets/sts3215_03a_no_horn_v1.stl"/>
-        </geometry>
-        <material name="sts3215"/>
+          <mesh filename="package://so_arm101_description/meshes/sts3215_03a_no_horn_v1.stl"/>
+        </geometry>
+        <material name="3d_printed"/>
       </visual>
       <collision>
         <origin xyz="8.32667e-17 -0.0424 0.0306" rpy="1.5708 1.5708 0"/>
         <geometry>
-          <mesh filename="package://so_arm100_description/SO101/assets/sts3215_03a_no_horn_v1.stl"/>
+          <mesh filename="package://so_arm101_description/meshes/sts3215_03a_no_horn_v1.stl"/>
         </geometry>
       </collision>
@@ -234,5 +234,5 @@
         <origin xyz="0 -0.028 0.0181" rpy="-1.5708 -1.5708 0"/>
         <geometry>
-          <mesh filename="package://so_arm100_description/SO101/assets/wrist_roll_pitch_so101_v2.stl"/>
+          <mesh filename="package://so_arm101_description/meshes/wrist_roll_pitch_so101_v2.stl"/>
         </geometry>
         <material name="3d_printed"/>
@@ -241,5 +241,5 @@
         <origin xyz="0 -0.028 0.0181" rpy="-1.5708 -1.5708 0"/>
         <geometry>
-          <mesh filename="package://so_arm100_description/SO101/assets/wrist_roll_pitch_so101_v2.stl"/>
+          <mesh filename="package://so_arm101_description/meshes/wrist_roll_pitch_so101_v2.stl"/>
         </geometry>
       </collision>
@@ -256,12 +256,12 @@
         <origin xyz="0.0077 0.0001 -0.0234" rpy="-1.5708 -5.19179e-17 -1.66533e-16"/>
         <geometry>
-          <mesh filename="package://so_arm100_description/SO101/assets/sts3215_03a_v1.stl"/>
-        </geometry>
-        <material name="sts3215"/>
+          <mesh filename="package://so_arm101_description/meshes/sts3215_03a_v1.stl"/>
+        </geometry>
+        <material name="3d_printed"/>
       </visual>
       <collision>
         <origin xyz="0.0077 0.0001 -0.0234" rpy="-1.5708 -5.19179e-17 -1.66533e-16"/>
         <geometry>
-          <mesh filename="package://so_arm100_description/SO101/assets/sts3215_03a_v1.stl"/>
+          <mesh filename="package://so_arm101_description/meshes/sts3215_03a_v1.stl"/>
         </geometry>
       </collision>
@@ -270,5 +270,5 @@
         <origin xyz="8.32667e-17 -0.000218214 0.000949706" rpy="-3.14159 -5.55112e-17 0"/>
         <geometry>
-          <mesh filename="package://so_arm100_description/SO101/assets/wrist_roll_follower_so101_v1.stl"/>
+          <mesh filename="package://so_arm101_description/meshes/wrist_roll_follower_so101_v1.stl"/>
         </geometry>
         <material name="3d_printed"/>
@@ -277,5 +277,5 @@
         <origin xyz="8.32667e-17 -0.000218214 0.000949706" rpy="-3.14159 -5.55112e-17 0"/>
         <geometry>
-          <mesh filename="package://so_arm100_description/SO101/assets/wrist_roll_follower_so101_v1.stl"/>
+          <mesh filename="package://so_arm101_description/meshes/wrist_roll_follower_so101_v1.stl"/>
         </geometry>
       </collision>
@@ -301,5 +301,5 @@
         <origin xyz="-5.55112e-17 -5.55112e-17 0.0189" rpy="9.53145e-17 6.93889e-18 1.24077e-24"/>
         <geometry>
-          <mesh filename="package://so_arm100_description/SO101/assets/moving_jaw_so101_v1.stl"/>
+          <mesh filename="package://so_arm101_description/meshes/moving_jaw_so101_v1.stl"/>
         </geometry>
         <material name="3d_printed"/>
@@ -308,5 +308,5 @@
         <origin xyz="-5.55112e-17 -5.55112e-17 0.0189" rpy="9.53145e-17 6.93889e-18 1.24077e-24"/>
         <geometry>
-          <mesh filename="package://so_arm100_description/SO101/assets/moving_jaw_so101_v1.stl"/>
+          <mesh filename="package://so_arm101_description/meshes/moving_jaw_so101_v1.stl"/>
         </geometry>
       </collision>
