Commit message: formats

File: so_arm100_description/urdf/so_arm100_macro.xacro (robot description, xacro)
@@ -26,7 +26,5 @@
       <visual>
         <geometry>
-          <mesh
-            filename="package://so_arm100_description/meshes/Base.stl"
-          />
+          <mesh filename="package://so_arm100_description/meshes/Base.stl" />
         </geometry>
         <material name="3d_printed" />
@@ -42,7 +40,5 @@
       <collision>
         <geometry>
-          <mesh
-            filename="package://so_arm100_description/meshes/Base.stl"
-          />
+          <mesh filename="package://so_arm100_description/meshes/Base.stl" />
         </geometry>
       </collision>

File: so_arm101_description/control/so_arm101.ros2_control.xacro (robot description, xacro)
@@ -16,5 +16,7 @@
         <xacro:if value="${ros2_control_hardware_type == 'mujoco'}">
           <plugin>mujoco_ros2_control/MujocoSystemInterface</plugin>
-          <param name="mujoco_model">$(find so_arm101_description)/mjcf/scene.xml</param>
+          <param name="mujoco_model">
+            $(find so_arm101_description)/mjcf/scene.xml
+          </param>
         </xacro:if>
       </hardware>

File: so_arm101_description/urdf/so_arm101_macro.xacro (robot description, xacro)
@@ -12,62 +12,109 @@
     <link name="${prefix}base_link">
       <inertial>
-        <origin xyz="0.0137179 -5.19711e-05 0.0334843" rpy="0 0 0"/>
-        <mass value="0.147"/>
-        <inertia ixx="0.000114686" ixy="-4.59787e-07" ixz="4.97151e-06" iyy="0.000136117" iyz="9.75275e-08" izz="0.000130364"/>
+        <origin xyz="0.0137179 -5.19711e-05 0.0334843" rpy="0 0 0" />
+        <mass value="0.147" />
+        <inertia
+          ixx="0.000114686"
+          ixy="-4.59787e-07"
+          ixz="4.97151e-06"
+          iyy="0.000136117"
+          iyz="9.75275e-08"
+          izz="0.000130364"
+        />
       </inertial>
       <!-- Part base_motor_holder_so101_v1 -->
       <visual>
-        <origin xyz="-0.00636471 -9.94414e-05 -0.0024" rpy="1.5708 -1.67685e-15 1.5708"/>
-        <geometry>
-          <mesh filename="package://so_arm101_description/meshes/base_motor_holder_so101_v1.stl"/>
-        </geometry>
-        <material name="3d_printed"/>
-      </visual>
-      <collision>
-        <origin xyz="-0.00636471 -9.94414e-05 -0.0024" rpy="1.5708 -1.67685e-15 1.5708"/>
-        <geometry>
-          <mesh filename="package://so_arm101_description/meshes/base_motor_holder_so101_v1.stl"/>
+        <origin
+          xyz="-0.00636471 -9.94414e-05 -0.0024"
+          rpy="1.5708 -1.67685e-15 1.5708"
+        />
+        <geometry>
+          <mesh
+            filename="package://so_arm101_description/meshes/base_motor_holder_so101_v1.stl"
+          />
+        </geometry>
+        <material name="3d_printed" />
+      </visual>
+      <collision>
+        <origin
+          xyz="-0.00636471 -9.94414e-05 -0.0024"
+          rpy="1.5708 -1.67685e-15 1.5708"
+        />
+        <geometry>
+          <mesh
+            filename="package://so_arm101_description/meshes/base_motor_holder_so101_v1.stl"
+          />
         </geometry>
       </collision>
       <!-- Part base_so101_v2 -->
       <visual>
-        <origin xyz="-0.00636471 -8.97657e-09 -0.0024" rpy="1.5708 -2.78073e-29 1.5708"/>
-        <geometry>
-          <mesh filename="package://so_arm101_description/meshes/base_so101_v2.stl"/>
-        </geometry>
-        <material name="3d_printed"/>
-      </visual>
-      <collision>
-        <origin xyz="-0.00636471 -8.97657e-09 -0.0024" rpy="1.5708 -2.78073e-29 1.5708"/>
-        <geometry>
-          <mesh filename="package://so_arm101_description/meshes/base_so101_v2.stl"/>
+        <origin
+          xyz="-0.00636471 -8.97657e-09 -0.0024"
+          rpy="1.5708 -2.78073e-29 1.5708"
+        />
+        <geometry>
+          <mesh
+            filename="package://so_arm101_description/meshes/base_so101_v2.stl"
+          />
+        </geometry>
+        <material name="3d_printed" />
+      </visual>
+      <collision>
+        <origin
+          xyz="-0.00636471 -8.97657e-09 -0.0024"
+          rpy="1.5708 -2.78073e-29 1.5708"
+        />
+        <geometry>
+          <mesh
+            filename="package://so_arm101_description/meshes/base_so101_v2.stl"
+          />
         </geometry>
       </collision>
       <!-- Part sts3215_03a_v1 -->
       <visual>
-        <origin xyz="0.0263353 -8.97657e-09 0.0437" rpy="-8.21148e-16 7.84513e-18 1.249e-15"/>
-        <geometry>
-          <mesh filename="package://so_arm101_description/meshes/sts3215_03a_v1.stl"/>
-        </geometry>
-        <material name="3d_printed"/>
-      </visual>
-      <collision>
-        <origin xyz="0.0263353 -8.97657e-09 0.0437" rpy="-8.21148e-16 7.84513e-18 1.249e-15"/>
-        <geometry>
-          <mesh filename="package://so_arm101_description/meshes/sts3215_03a_v1.stl"/>
+        <origin
+          xyz="0.0263353 -8.97657e-09 0.0437"
+          rpy="-8.21148e-16 7.84513e-18 1.249e-15"
+        />
+        <geometry>
+          <mesh
+            filename="package://so_arm101_description/meshes/sts3215_03a_v1.stl"
+          />
+        </geometry>
+        <material name="3d_printed" />
+      </visual>
+      <collision>
+        <origin
+          xyz="0.0263353 -8.97657e-09 0.0437"
+          rpy="-8.21148e-16 7.84513e-18 1.249e-15"
+        />
+        <geometry>
+          <mesh
+            filename="package://so_arm101_description/meshes/sts3215_03a_v1.stl"
+          />
         </geometry>
       </collision>
       <!-- Part waveshare_mounting_plate_so101_v2 -->
       <visual>
-        <origin xyz="-0.0309827 -0.000199441 0.0474" rpy="1.5708 -1.35493e-14 1.5708"/>
-        <geometry>
-          <mesh filename="package://so_arm101_description/meshes/waveshare_mounting_plate_so101_v2.stl"/>
-        </geometry>
-        <material name="3d_printed"/>
-      </visual>
-      <collision>
-        <origin xyz="-0.0309827 -0.000199441 0.0474" rpy="1.5708 -1.35493e-14 1.5708"/>
-        <geometry>
-          <mesh filename="package://so_arm101_description/meshes/waveshare_mounting_plate_so101_v2.stl"/>
+        <origin
+          xyz="-0.0309827 -0.000199441 0.0474"
+          rpy="1.5708 -1.35493e-14 1.5708"
+        />
+        <geometry>
+          <mesh
+            filename="package://so_arm101_description/meshes/waveshare_mounting_plate_so101_v2.stl"
+          />
+        </geometry>
+        <material name="3d_printed" />
+      </visual>
+      <collision>
+        <origin
+          xyz="-0.0309827 -0.000199441 0.0474"
+          rpy="1.5708 -1.35493e-14 1.5708"
+        />
+        <geometry>
+          <mesh
+            filename="package://so_arm101_description/meshes/waveshare_mounting_plate_so101_v2.stl"
+          />
         </geometry>
       </collision>
@@ -76,48 +123,79 @@
     <link name="${prefix}shoulder_link">
       <inertial>
-        <origin xyz="-0.0307604 -1.66727e-05 -0.0252713" rpy="0 0 0"/>
-        <mass value="0.100006"/>
-        <inertia ixx="8.3759e-05" ixy="7.55525e-08" ixz="-1.16342e-06" iyy="8.10403e-05" iyz="1.54663e-07" izz="2.39783e-05"/>
+        <origin xyz="-0.0307604 -1.66727e-05 -0.0252713" rpy="0 0 0" />
+        <mass value="0.100006" />
+        <inertia
+          ixx="8.3759e-05"
+          ixy="7.55525e-08"
+          ixz="-1.16342e-06"
+          iyy="8.10403e-05"
+          iyz="1.54663e-07"
+          izz="2.39783e-05"
+        />
       </inertial>
       <!-- Part sts3215_03a_v1_2 -->
       <visual>
-        <origin xyz="-0.0303992 0.000422241 -0.0417" rpy="1.5708 1.5708 0"/>
-        <geometry>
-          <mesh filename="package://so_arm101_description/meshes/sts3215_03a_v1.stl"/>
-        </geometry>
-        <material name="3d_printed"/>
-      </visual>
-      <collision>
-        <origin xyz="-0.0303992 0.000422241 -0.0417" rpy="1.5708 1.5708 0"/>
-        <geometry>
-          <mesh filename="package://so_arm101_description/meshes/sts3215_03a_v1.stl"/>
+        <origin xyz="-0.0303992 0.000422241 -0.0417" rpy="1.5708 1.5708 0" />
+        <geometry>
+          <mesh
+            filename="package://so_arm101_description/meshes/sts3215_03a_v1.stl"
+          />
+        </geometry>
+        <material name="3d_printed" />
+      </visual>
+      <collision>
+        <origin xyz="-0.0303992 0.000422241 -0.0417" rpy="1.5708 1.5708 0" />
+        <geometry>
+          <mesh
+            filename="package://so_arm101_description/meshes/sts3215_03a_v1.stl"
+          />
         </geometry>
       </collision>
       <!-- Part motor_holder_so101_base_v1 -->
       <visual>
-        <origin xyz="-0.0675992 -0.000177759 0.0158499" rpy="1.5708 -1.5708 0"/>
-        <geometry>
-          <mesh filename="package://so_arm101_description/meshes/motor_holder_so101_base_v1.stl"/>
-        </geometry>
-        <material name="3d_printed"/>
-      </visual>
-      <collision>
-        <origin xyz="-0.0675992 -0.000177759 0.0158499" rpy="1.5708 -1.5708 0"/>
-        <geometry>
-          <mesh filename="package://so_arm101_description/meshes/motor_holder_so101_base_v1.stl"/>
+        <origin
+          xyz="-0.0675992 -0.000177759 0.0158499"
+          rpy="1.5708 -1.5708 0"
+        />
+        <geometry>
+          <mesh
+            filename="package://so_arm101_description/meshes/motor_holder_so101_base_v1.stl"
+          />
+        </geometry>
+        <material name="3d_printed" />
+      </visual>
+      <collision>
+        <origin
+          xyz="-0.0675992 -0.000177759 0.0158499"
+          rpy="1.5708 -1.5708 0"
+        />
+        <geometry>
+          <mesh
+            filename="package://so_arm101_description/meshes/motor_holder_so101_base_v1.stl"
+          />
         </geometry>
       </collision>
       <!-- Part rotation_pitch_so101_v1 -->
       <visual>
-        <origin xyz="0.0122008 2.22413e-05 0.0464" rpy="-1.5708 2.35221e-33 0"/>
-        <geometry>
-          <mesh filename="package://so_arm101_description/meshes/rotation_pitch_so101_v1.stl"/>
-        </geometry>
-        <material name="3d_printed"/>
-      </visual>
-      <collision>
-        <origin xyz="0.0122008 2.22413e-05 0.0464" rpy="-1.5708 2.35221e-33 0"/>
-        <geometry>
-          <mesh filename="package://so_arm101_description/meshes/rotation_pitch_so101_v1.stl"/>
+        <origin
+          xyz="0.0122008 2.22413e-05 0.0464"
+          rpy="-1.5708 2.35221e-33 0"
+        />
+        <geometry>
+          <mesh
+            filename="package://so_arm101_description/meshes/rotation_pitch_so101_v1.stl"
+          />
+        </geometry>
+        <material name="3d_printed" />
+      </visual>
+      <collision>
+        <origin
+          xyz="0.0122008 2.22413e-05 0.0464"
+          rpy="-1.5708 2.35221e-33 0"
+        />
+        <geometry>
+          <mesh
+            filename="package://so_arm101_description/meshes/rotation_pitch_so101_v1.stl"
+          />
         </geometry>
       </collision>
@@ -126,34 +204,55 @@
     <link name="${prefix}upper_arm_link">
       <inertial>
-        <origin xyz="-0.0898471 -0.00838224 0.0184089" rpy="0 0 0"/>
-        <mass value="0.103"/>
-        <inertia ixx="4.08002e-05" ixy="-1.97819e-05" ixz="-4.03016e-08" iyy="0.000147318" iyz="8.97326e-09" izz="0.000142487"/>
+        <origin xyz="-0.0898471 -0.00838224 0.0184089" rpy="0 0 0" />
+        <mass value="0.103" />
+        <inertia
+          ixx="4.08002e-05"
+          ixy="-1.97819e-05"
+          ixz="-4.03016e-08"
+          iyy="0.000147318"
+          iyz="8.97326e-09"
+          izz="0.000142487"
+        />
       </inertial>
       <!-- Part sts3215_03a_v1_3 -->
       <visual>
-        <origin xyz="-0.11257 -0.0155 0.0187" rpy="-3.14159 -5.27356e-16 -1.5708"/>
-        <geometry>
-          <mesh filename="package://so_arm101_description/meshes/sts3215_03a_v1.stl"/>
-        </geometry>
-        <material name="3d_printed"/>
-      </visual>
-      <collision>
-        <origin xyz="-0.11257 -0.0155 0.0187" rpy="-3.14159 -5.27356e-16 -1.5708"/>
-        <geometry>
-          <mesh filename="package://so_arm101_description/meshes/sts3215_03a_v1.stl"/>
+        <origin
+          xyz="-0.11257 -0.0155 0.0187"
+          rpy="-3.14159 -5.27356e-16 -1.5708"
+        />
+        <geometry>
+          <mesh
+            filename="package://so_arm101_description/meshes/sts3215_03a_v1.stl"
+          />
+        </geometry>
+        <material name="3d_printed" />
+      </visual>
+      <collision>
+        <origin
+          xyz="-0.11257 -0.0155 0.0187"
+          rpy="-3.14159 -5.27356e-16 -1.5708"
+        />
+        <geometry>
+          <mesh
+            filename="package://so_arm101_description/meshes/sts3215_03a_v1.stl"
+          />
         </geometry>
       </collision>
       <!-- Part upper_arm_so101_v1 -->
       <visual>
-        <origin xyz="-0.065085 0.012 0.0182" rpy="3.14159 -0 -1.30911e-30"/>
-        <geometry>
-          <mesh filename="package://so_arm101_description/meshes/upper_arm_so101_v1.stl"/>
-        </geometry>
-        <material name="3d_printed"/>
-      </visual>
-      <collision>
-        <origin xyz="-0.065085 0.012 0.0182" rpy="3.14159 -0 -1.30911e-30"/>
-        <geometry>
-          <mesh filename="package://so_arm101_description/meshes/upper_arm_so101_v1.stl"/>
+        <origin xyz="-0.065085 0.012 0.0182" rpy="3.14159 -0 -1.30911e-30" />
+        <geometry>
+          <mesh
+            filename="package://so_arm101_description/meshes/upper_arm_so101_v1.stl"
+          />
+        </geometry>
+        <material name="3d_printed" />
+      </visual>
+      <collision>
+        <origin xyz="-0.065085 0.012 0.0182" rpy="3.14159 -0 -1.30911e-30" />
+        <geometry>
+          <mesh
+            filename="package://so_arm101_description/meshes/upper_arm_so101_v1.stl"
+          />
         </geometry>
       </collision>
@@ -162,48 +261,79 @@
     <link name="${prefix}lower_arm_link">
       <inertial>
-        <origin xyz="-0.0980701 0.00324376 0.0182831" rpy="0 0 0"/>
-        <mass value="0.104"/>
-        <inertia ixx="2.87438e-05" ixy="7.41152e-06" ixz="1.26409e-06" iyy="0.000159844" iyz="-4.90188e-08" izz="0.00014529"/>
+        <origin xyz="-0.0980701 0.00324376 0.0182831" rpy="0 0 0" />
+        <mass value="0.104" />
+        <inertia
+          ixx="2.87438e-05"
+          ixy="7.41152e-06"
+          ixz="1.26409e-06"
+          iyy="0.000159844"
+          iyz="-4.90188e-08"
+          izz="0.00014529"
+        />
       </inertial>
       <!-- Part under_arm_so101_v1 -->
       <visual>
-        <origin xyz="-0.0648499 -0.032 0.0182" rpy="3.14159 -0 6.67202e-31"/>
-        <geometry>
-          <mesh filename="package://so_arm101_description/meshes/under_arm_so101_v1.stl"/>
-        </geometry>
-        <material name="3d_printed"/>
-      </visual>
-      <collision>
-        <origin xyz="-0.0648499 -0.032 0.0182" rpy="3.14159 -0 6.67202e-31"/>
-        <geometry>
-          <mesh filename="package://so_arm101_description/meshes/under_arm_so101_v1.stl"/>
+        <origin xyz="-0.0648499 -0.032 0.0182" rpy="3.14159 -0 6.67202e-31" />
+        <geometry>
+          <mesh
+            filename="package://so_arm101_description/meshes/under_arm_so101_v1.stl"
+          />
+        </geometry>
+        <material name="3d_printed" />
+      </visual>
+      <collision>
+        <origin xyz="-0.0648499 -0.032 0.0182" rpy="3.14159 -0 6.67202e-31" />
+        <geometry>
+          <mesh
+            filename="package://so_arm101_description/meshes/under_arm_so101_v1.stl"
+          />
         </geometry>
       </collision>
       <!-- Part motor_holder_so101_wrist_v1 -->
       <visual>
-        <origin xyz="-0.0648499 -0.032 0.018" rpy="-3.14159 -2.55351e-15 -1.83387e-30"/>
-        <geometry>
-          <mesh filename="package://so_arm101_description/meshes/motor_holder_so101_wrist_v1.stl"/>
-        </geometry>
-        <material name="3d_printed"/>
-      </visual>
-      <collision>
-        <origin xyz="-0.0648499 -0.032 0.018" rpy="-3.14159 -2.55351e-15 -1.83387e-30"/>
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
Commit message: Adds SO-ARM101 support and removes submodule (#30)

File: so_arm100_description/urdf/so_arm100_macro.xacro (robot description, xacro)
@@ -26,23 +26,19 @@
       <visual>
         <geometry>
-          <mesh
-            filename="package://so_arm100_description/SO100/assets/Base.stl"
-          />
-        </geometry>
-        <material name="3d_printed" />
-      </visual>
-      <visual>
-        <geometry>
-          <mesh
-            filename="package://so_arm100_description/SO100/assets/Base_Motor.stl"
-          />
-        </geometry>
-        <material name="sts3215" />
-      </visual>
-      <collision>
-        <geometry>
-          <mesh
-            filename="package://so_arm100_description/SO100/assets/Base.stl"
-          />
+          <mesh filename="package://so_arm100_description/meshes/Base.stl" />
+        </geometry>
+        <material name="3d_printed" />
+      </visual>
+      <visual>
+        <geometry>
+          <mesh
+            filename="package://so_arm100_description/meshes/Base_Motor.stl"
+          />
+        </geometry>
+        <material name="sts3215" />
+      </visual>
+      <collision>
+        <geometry>
+          <mesh filename="package://so_arm100_description/meshes/Base.stl" />
         </geometry>
       </collision>
@@ -65,21 +61,21 @@
         <geometry>
           <mesh
-            filename="package://so_arm100_description/SO100/assets/Rotation_Pitch.stl"
-          />
-        </geometry>
-        <material name="3d_printed" />
-      </visual>
-      <visual>
-        <geometry>
-          <mesh
-            filename="package://so_arm100_description/SO100/assets/Rotation_Pitch_Motor.stl"
-          />
-        </geometry>
-        <material name="sts3215" />
-      </visual>
-      <collision>
-        <geometry>
-          <mesh
-            filename="package://so_arm100_description/SO100/assets/Rotation_Pitch.stl"
+            filename="package://so_arm100_description/meshes/Rotation_Pitch.stl"
+          />
+        </geometry>
+        <material name="3d_printed" />
+      </visual>
+      <visual>
+        <geometry>
+          <mesh
+            filename="package://so_arm100_description/meshes/Rotation_Pitch_Motor.stl"
+          />
+        </geometry>
+        <material name="sts3215" />
+      </visual>
+      <collision>
+        <geometry>
+          <mesh
+            filename="package://so_arm100_description/meshes/Rotation_Pitch.stl"
           />
         </geometry>
@@ -103,21 +99,21 @@
         <geometry>
           <mesh
-            filename="package://so_arm100_description/SO100/assets/Upper_Arm.stl"
-          />
-        </geometry>
-        <material name="3d_printed" />
-      </visual>
-      <visual>
-        <geometry>
-          <mesh
-            filename="package://so_arm100_description/SO100/assets/Upper_Arm_Motor.stl"
-          />
-        </geometry>
-        <material name="sts3215" />
-      </visual>
-      <collision>
-        <geometry>
-          <mesh
-            filename="package://so_arm100_description/SO100/assets/Upper_Arm.stl"
+            filename="package://so_arm100_description/meshes/Upper_Arm.stl"
+          />
+        </geometry>
+        <material name="3d_printed" />
+      </visual>
+      <visual>
+        <geometry>
+          <mesh
+            filename="package://so_arm100_description/meshes/Upper_Arm_Motor.stl"
+          />
+        </geometry>
+        <material name="sts3215" />
+      </visual>
+      <collision>
+        <geometry>
+          <mesh
+            filename="package://so_arm100_description/meshes/Upper_Arm.stl"
           />
         </geometry>
@@ -141,21 +137,21 @@
         <geometry>
           <mesh
-            filename="package://so_arm100_description/SO100/assets/Lower_Arm.stl"
-          />
-        </geometry>
-        <material name="3d_printed" />
-      </visual>
-      <visual>
-        <geometry>
-          <mesh
-            filename="package://so_arm100_description/SO100/assets/Lower_Arm_Motor.stl"
-          />
-        </geometry>
-        <material name="sts3215" />
-      </visual>
-      <collision>
-        <geometry>
-          <mesh
-            filename="package://so_arm100_description/SO100/assets/Lower_Arm.stl"
+            filename="package://so_arm100_description/meshes/Lower_Arm.stl"
+          />
+        </geometry>
+        <material name="3d_printed" />
+      </visual>
+      <visual>
+        <geometry>
+          <mesh
+            filename="package://so_arm100_description/meshes/Lower_Arm_Motor.stl"
+          />
+        </geometry>
+        <material name="sts3215" />
+      </visual>
+      <collision>
+        <geometry>
+          <mesh
+            filename="package://so_arm100_description/meshes/Lower_Arm.stl"
           />
         </geometry>
@@ -179,21 +175,21 @@
         <geometry>
           <mesh
-            filename="package://so_arm100_description/SO100/assets/Wrist_Pitch_Roll.stl"
-          />
-        </geometry>
-        <material name="3d_printed" />
-      </visual>
-      <visual>
-        <geometry>
-          <mesh
-            filename="package://so_arm100_description/SO100/assets/Wrist_Pitch_Roll_Motor.stl"
-          />
-        </geometry>
-        <material name="sts3215" />
-      </visual>
-      <collision>
-        <geometry>
-          <mesh
-            filename="package://so_arm100_description/SO100/assets/Wrist_Pitch_Roll.stl"
+            filename="package://so_arm100_description/meshes/Wrist_Pitch_Roll.stl"
+          />
+        </geometry>
+        <material name="3d_printed" />
+      </visual>
+      <visual>
+        <geometry>
+          <mesh
+            filename="package://so_arm100_description/meshes/Wrist_Pitch_Roll_Motor.stl"
+          />
+        </geometry>
+        <material name="sts3215" />
+      </visual>
+      <collision>
+        <geometry>
+          <mesh
+            filename="package://so_arm100_description/meshes/Wrist_Pitch_Roll.stl"
           />
         </geometry>
@@ -217,13 +213,13 @@
         <geometry>
           <mesh
-            filename="package://so_arm100_description/SO100/assets/Fixed_Jaw.stl"
-          />
-        </geometry>
-        <material name="3d_printed" />
-      </visual>
-      <visual>
-        <geometry>
-          <mesh
-            filename="package://so_arm100_description/SO100/assets/Fixed_Jaw_Motor.stl"
+            filename="package://so_arm100_description/meshes/Fixed_Jaw.stl"
+          />
+        </geometry>
+        <material name="3d_printed" />
+      </visual>
+      <visual>
+        <geometry>
+          <mesh
+            filename="package://so_arm100_description/meshes/Fixed_Jaw_Motor.stl"
           />
         </geometry>
@@ -248,5 +244,5 @@
         <geometry>
           <mesh
-            filename="package://so_arm100_description/SO100/assets/Moving_Jaw.stl"
+            filename="package://so_arm100_description/meshes/Moving_Jaw.stl"
           />
         </geometry>
