Commit message: Get so_arm_gz_bringup to work with both arms
Signed-off-by: Yadunund Vijay <yadunund@gmail.com>

File: so_arm100_description/urdf/so_arm100_macro.xacro (robot description, xacro)
@@ -16,4 +16,12 @@
       <color rgba="0.1 0.1 0.1 1.0" />
     </material>
+    <!-- World link (fixed reference for Gazebo) -->
+    <link name="world" />
+    <!-- Fixed joint from world to base -->
+    <joint name="${prefix}world_to_base_joint" type="fixed">
+      <origin xyz="0 0 0" rpy="0 0 0" />
+      <parent link="world" />
+      <child link="${prefix}base_link" />
+    </joint>
     <!-- Link base -->
     <link name="${prefix}base_link">

File: so_arm101_description/control/so_arm101.ros2_control.xacro (robot description, xacro)
@@ -19,4 +19,7 @@
             $(find so_arm101_description)/mjcf/scene.xml
           </param>
+        </xacro:if>
+        <xacro:if value="${ros2_control_hardware_type == 'gazebo'}">
+          <plugin>gz_ros2_control/GazeboSimSystem</plugin>
         </xacro:if>
       </hardware>

File: so_arm101_description/urdf/so_arm101.urdf.xacro (robot description, xacro)
@@ -16,4 +16,7 @@
   <xacro:include filename="$(arg urdf_file)" />
   <xacro:so_arm101 prefix="$(arg prefix)" color="$(arg color)" />
+  <!-- parameters -->
+  <xacro:arg name="simulation_controllers" default="" />
+  <xacro:arg name="ros_namespace" default="" />
   <!-- ros2_control description -->
   <xacro:include filename="$(arg ros2_control_file)" />
@@ -23,3 +26,13 @@
     usb_port="$(arg usb_port)"
   />
+  <gazebo reference="world">
+  </gazebo>
+  <gazebo>
+    <plugin filename="gz_ros2_control-system" name="gz_ros2_control::GazeboSimROS2ControlPlugin">
+      <parameters>$(arg simulation_controllers)</parameters>
+      <ros>
+        <namespace>$(arg ros_namespace)</namespace>
+      </ros>
+    </plugin>
+  </gazebo>
 </robot>

File: so_arm101_description/urdf/so_arm101_macro.xacro (robot description, xacro)
@@ -9,4 +9,12 @@
       <color rgba="0.1 0.1 0.1 1.0" />
     </material>
+    <!-- World link (fixed reference for Gazebo) -->
+    <link name="world" />
+    <!-- Fixed joint from world to base -->
+    <joint name="${prefix}world_to_base_joint" type="fixed">
+      <origin xyz="0 0 0" rpy="0 0 0" />
+      <parent link="world" />
+      <child link="${prefix}base_link" />
+    </joint>
     <!-- Link base -->
     <link name="${prefix}base_link">

Commit message: Formatting

File: so_arm100_description/urdf/so_arm100_macro.xacro (robot description, xacro)
@@ -8,6 +8,7 @@
 -->
 <robot xmlns:xacro="http://ros.org/wiki/xacro">
-  <xacro:macro name="so_arm100"
-               params="prefix
+  <xacro:macro
+    name="so_arm100"
+    params="prefix
                        color:='1.0 0.82 0.12 1.0'
                        parent:=world
@@ -17,5 +18,6 @@
                        roll:=0.0
                        pitch:=0.0
-                       yaw:=0.0">
+                       yaw:=0.0"
+  >
     <!-- Materials -->
     <material name="3d_printed">

File: so_arm101_description/urdf/so_arm101_macro.xacro (robot description, xacro)
@@ -1,6 +1,7 @@
 <?xml version="1.0" encoding="utf-8" ?>
 <robot xmlns:xacro="http://ros.org/wiki/xacro">
-  <xacro:macro name="so_arm101"
-               params="prefix
+  <xacro:macro
+    name="so_arm101"
+    params="prefix
                        color:='1.0 0.82 0.12 1.0'
                        parent:=world
@@ -10,5 +11,6 @@
                        roll:=0.0
                        pitch:=0.0
-                       yaw:=0.0">
+                       yaw:=0.0"
+  >
     <!-- Materials -->
     <material name="3d_printed">

Commit message: Add pose and parent args to xacros (#31)

File: so_arm100_description/urdf/so_arm100_macro.xacro (robot description, xacro)
@@ -8,5 +8,17 @@
 -->
 <robot xmlns:xacro="http://ros.org/wiki/xacro">
-  <xacro:macro name="so_arm100" params="prefix color:='1.0 0.82 0.12 1.0'">
+  <xacro:macro
+    name="so_arm100"
+    params="
+      prefix
+      color:='1.0 0.82 0.12 1.0'
+      parent:=world
+      x:=0.0
+      y:=0.0
+      z:=0.0
+      roll:=0.0
+      pitch:=0.0
+      yaw:=0.0"
+  >
     <!-- Materials -->
     <material name="3d_printed">
@@ -16,10 +28,8 @@
       <color rgba="0.1 0.1 0.1 1.0" />
     </material>
-    <!-- World link (fixed reference for Gazebo) -->
-    <link name="world" />
-    <!-- Fixed joint from world to base -->
-    <joint name="${prefix}world_to_base_joint" type="fixed">
-      <origin xyz="0 0 0" rpy="0 0 0" />
-      <parent link="world" />
+    <!-- Fixed joint from parent to base -->
+    <joint name="${prefix}${parent}_to_base_joint" type="fixed">
+      <origin xyz="${x} ${y} ${z}" rpy="${roll} ${pitch} ${yaw}" />
+      <parent link="${parent}" />
       <child link="${prefix}base_link" />
     </joint>

File: so_arm101_description/urdf/so_arm101_macro.xacro (robot description, xacro)
@@ -1,5 +1,17 @@
 <?xml version="1.0" encoding="utf-8" ?>
 <robot xmlns:xacro="http://ros.org/wiki/xacro">
-  <xacro:macro name="so_arm101" params="prefix color:='0.2 0.7 0.85 1.0'">
+  <xacro:macro
+    name="so_arm101"
+    params="
+      prefix
+      color:='1.0 0.82 0.12 1.0'
+      parent:=world
+      x:=0.0
+      y:=0.0
+      z:=0.0
+      roll:=0.0
+      pitch:=0.0
+      yaw:=0.0"
+  >
     <!-- Materials -->
     <material name="3d_printed">
@@ -9,10 +21,8 @@
       <color rgba="0.1 0.1 0.1 1.0" />
     </material>
-    <!-- World link (fixed reference for Gazebo) -->
-    <link name="world" />
-    <!-- Fixed joint from world to base -->
-    <joint name="${prefix}world_to_base_joint" type="fixed">
-      <origin xyz="0 0 0" rpy="0 0 0" />
-      <parent link="world" />
+    <!-- Fixed joint from parent to base -->
+    <joint name="${prefix}${parent}_to_base_joint" type="fixed">
+      <origin xyz="${x} ${y} ${z}" rpy="${roll} ${pitch} ${yaw}" />
+      <parent link="${parent}" />
       <child link="${prefix}base_link" />
     </joint>
