Commit message: Configure xacro via launch args
Signed-off-by: Yadunund <yadunund@gmail.com>

File: so_arm100_description/control/so_arm100.ros2_control.xacro (robot description, xacro)
@@ -1,5 +1,5 @@
 <?xml version="1.0" ?>
 <robot xmlns:xacro="http://www.ros.org/wiki/xacro">
-  <xacro:macro name="ros2_control" params="ros2_control_hardware_type">
+  <xacro:macro name="ros2_control" params="ros2_control_hardware_type usb_port">
     <ros2_control name="SO-ARM100" type="system">
       <hardware>
@@ -9,5 +9,5 @@
         <xacro:if value="${ros2_control_hardware_type == 'real'}">
           <plugin>feetech_ros2_driver/FeetechHardwareInterface</plugin>
-          <param name="usb_port">/dev/LeRobotFollower</param>
+          <param name="usb_port">${usb_port}</param>
         </xacro:if>
       </hardware>

File: so_arm100_description/urdf/so_arm100.urdf.xacro (robot description, xacro)
@@ -2,10 +2,12 @@
 <robot xmlns:xacro="http://www.ros.org/wiki/xacro" name="so_100arm">
   <xacro:arg name="ros2_control_hardware_type" default="mock_components" />
-  <xacro:include filename="so_arm100.urdf" />
-  <xacro:include
-    filename="$(find so_arm100_description)/control/so_arm100.ros2_control.xacro"
-  />
+  <xacro:arg name="ros2_control_file" default="$(find so_arm100_description)/control/so_arm100.ros2_control.xacro" />
+  <xacro:arg name="urdf_file" default="$(find so_arm100_description)/urdf/so_arm100.urdf" />
+  <xacro:arg name="usb_port" default="/dev/LeRobotFollower" />
+  <xacro:include filename="$(arg urdf_file)" />
+  <xacro:include filename="$(arg ros2_control_file)" />
   <xacro:ros2_control
     ros2_control_hardware_type="$(arg ros2_control_hardware_type)"
+    usb_port="$(arg usb_port)"
   />
 </robot>

Commit message: Allow robot links and joints to be namespaced
Signed-off-by: Yadunund <yadunund@gmail.com>

File: so_arm100_description/control/so_arm100.ros2_control.xacro (robot description, xacro)
@@ -1,5 +1,5 @@
 <?xml version="1.0" ?>
 <robot xmlns:xacro="http://www.ros.org/wiki/xacro">
-  <xacro:macro name="ros2_control" params="ros2_control_hardware_type usb_port">
+  <xacro:macro name="ros2_control" params="prefix ros2_control_hardware_type usb_port">
     <ros2_control name="SO-ARM100" type="system">
       <hardware>
@@ -12,5 +12,5 @@
         </xacro:if>
       </hardware>
-      <joint name="shoulder_pan_joint">
+      <joint name="${prefix}shoulder_pan_joint">
         <param name="initial_position">0.0</param>
         <param name="id">1</param>
@@ -21,5 +21,5 @@
         <state_interface name="velocity" />
       </joint>
-      <joint name="shoulder_lift_joint">
+      <joint name="${prefix}shoulder_lift_joint">
         <param name="id">2</param>
         <param name="p_cofficient">16</param>
@@ -30,5 +30,5 @@
         <state_interface name="velocity" />
       </joint>
-      <joint name="elbow_joint">
+      <joint name="${prefix}elbow_joint">
         <param name="id">3</param>
         <param name="offset">2080</param>
@@ -39,5 +39,5 @@
         <state_interface name="velocity" />
       </joint>
-      <joint name="wrist_pitch_joint">
+      <joint name="${prefix}wrist_pitch_joint">
         <param name="id">4</param>
         <param name="offset">3110</param>
@@ -48,5 +48,5 @@
         <state_interface name="velocity" />
       </joint>
-      <joint name="wrist_roll_joint">
+      <joint name="${prefix}wrist_roll_joint">
         <param name="id">5</param>
         <param name="offset">1024</param>
@@ -57,5 +57,5 @@
         <state_interface name="velocity" />
       </joint>
-      <joint name="jaw_joint">
+      <joint name="${prefix}jaw_joint">
         <param name="id">6</param>
         <param name="offset">2070</param>

File: so_arm100_description/urdf/so_arm100.urdf.xacro (robot description, xacro)
@@ -3,9 +3,14 @@
   <xacro:arg name="ros2_control_hardware_type" default="mock_components" />
   <xacro:arg name="ros2_control_file" default="$(find so_arm100_description)/control/so_arm100.ros2_control.xacro" />
-  <xacro:arg name="urdf_file" default="$(find so_arm100_description)/urdf/so_arm100.urdf" />
+  <xacro:arg name="urdf_file" default="$(find so_arm100_description)/urdf/so_arm100_macro.xacro" />
   <xacro:arg name="usb_port" default="/dev/LeRobotFollower" />
+  <xacro:arg name="prefix" default="" />
+  <!-- Robot description -->
   <xacro:include filename="$(arg urdf_file)" />
+  <xacro:so_arm100 prefix="$(arg prefix)"/>
+  <!-- ros2_control description -->
   <xacro:include filename="$(arg ros2_control_file)" />
   <xacro:ros2_control
+    prefix="$(arg prefix)"
     ros2_control_hardware_type="$(arg ros2_control_hardware_type)"
     usb_port="$(arg usb_port)"

Commit message: Pre-commit

File: so_arm100_description/control/so_arm100.ros2_control.xacro (robot description, xacro)
@@ -1,5 +1,8 @@
 <?xml version="1.0" ?>
 <robot xmlns:xacro="http://www.ros.org/wiki/xacro">
-  <xacro:macro name="ros2_control" params="prefix ros2_control_hardware_type usb_port">
+  <xacro:macro
+    name="ros2_control"
+    params="prefix ros2_control_hardware_type usb_port"
+  >
     <ros2_control name="SO-ARM100" type="system">
       <hardware>

File: so_arm100_description/urdf/so_arm100.urdf.xacro (robot description, xacro)
@@ -2,11 +2,17 @@
 <robot xmlns:xacro="http://www.ros.org/wiki/xacro" name="so_100arm">
   <xacro:arg name="ros2_control_hardware_type" default="mock_components" />
-  <xacro:arg name="ros2_control_file" default="$(find so_arm100_description)/control/so_arm100.ros2_control.xacro" />
-  <xacro:arg name="urdf_file" default="$(find so_arm100_description)/urdf/so_arm100_macro.xacro" />
+  <xacro:arg
+    name="ros2_control_file"
+    default="$(find so_arm100_description)/control/so_arm100.ros2_control.xacro"
+  />
+  <xacro:arg
+    name="urdf_file"
+    default="$(find so_arm100_description)/urdf/so_arm100_macro.xacro"
+  />
   <xacro:arg name="usb_port" default="/dev/LeRobotFollower" />
   <xacro:arg name="prefix" default="" />
   <!-- Robot description -->
   <xacro:include filename="$(arg urdf_file)" />
-  <xacro:so_arm100 prefix="$(arg prefix)"/>
+  <xacro:so_arm100 prefix="$(arg prefix)" />
   <!-- ros2_control description -->
   <xacro:include filename="$(arg ros2_control_file)" />

File: so_arm100_description/urdf/so_arm100_macro.xacro (robot description, xacro)
@@ -45,5 +45,7 @@
         </geometry>
         <material name="">
-          <color rgba="0.792156862745098 0.819607843137255 0.933333333333333 1" />
+          <color
+            rgba="0.792156862745098 0.819607843137255 0.933333333333333 1"
+          />
         </material>
       </visual>
@@ -79,5 +81,7 @@
         </geometry>
         <material name="">
-          <color rgba="0.792156862745098 0.819607843137255 0.933333333333333 1" />
+          <color
+            rgba="0.792156862745098 0.819607843137255 0.933333333333333 1"
+          />
         </material>
       </visual>
@@ -117,14 +121,20 @@
         <origin xyz="0 0 0" rpy="0 0 0" />
         <geometry>
-          <mesh filename="package://so_arm100_description/meshes/Upper_Arm.STL" />
-        </geometry>
-        <material name="">
-          <color rgba="0.792156862745098 0.819607843137255 0.933333333333333 1" />
-        </material>
-      </visual>
-      <collision>
-        <origin xyz="0 0 0" rpy="0 0 0" />
-        <geometry>
-          <mesh filename="package://so_arm100_description/meshes/Upper_Arm.STL" />
+          <mesh
+            filename="package://so_arm100_description/meshes/Upper_Arm.STL"
+          />
+        </geometry>
+        <material name="">
+          <color
+            rgba="0.792156862745098 0.819607843137255 0.933333333333333 1"
+          />
+        </material>
+      </visual>
+      <collision>
+        <origin xyz="0 0 0" rpy="0 0 0" />
+        <geometry>
+          <mesh
+            filename="package://so_arm100_description/meshes/Upper_Arm.STL"
+          />
         </geometry>
       </collision>
@@ -156,14 +166,20 @@
         <origin xyz="0 0 0" rpy="0 0 0" />
         <geometry>
-          <mesh filename="package://so_arm100_description/meshes/Lower_Arm.STL" />
-        </geometry>
-        <material name="">
-          <color rgba="0.792156862745098 0.819607843137255 0.933333333333333 1" />
-        </material>
-      </visual>
-      <collision>
-        <origin xyz="0 0 0" rpy="0 0 0" />
-        <geometry>
-          <mesh filename="package://so_arm100_description/meshes/Lower_Arm.STL" />
+          <mesh
+            filename="package://so_arm100_description/meshes/Lower_Arm.STL"
+          />
+        </geometry>
+        <material name="">
+          <color
+            rgba="0.792156862745098 0.819607843137255 0.933333333333333 1"
+          />
+        </material>
+      </visual>
+      <collision>
+        <origin xyz="0 0 0" rpy="0 0 0" />
+        <geometry>
+          <mesh
+            filename="package://so_arm100_description/meshes/Lower_Arm.STL"
+          />
         </geometry>
       </collision>
@@ -200,5 +216,7 @@
         </geometry>
         <material name="">
-          <color rgba="0.792156862745098 0.819607843137255 0.933333333333333 1" />
+          <color
+            rgba="0.792156862745098 0.819607843137255 0.933333333333333 1"
+          />
         </material>
       </visual>
@@ -238,14 +256,20 @@
         <origin xyz="0 0 0" rpy="0 0 0" />
         <geometry>
-          <mesh filename="package://so_arm100_description/meshes/Fixed_Jaw.STL" />
-        </geometry>
-        <material name="">
-          <color rgba="0.792156862745098 0.819607843137255 0.933333333333333 1" />
-        </material>
-      </visual>
-      <collision>
-        <origin xyz="0 0 0" rpy="0 0 0" />
-        <geometry>
-          <mesh filename="package://so_arm100_description/meshes/Fixed_Jaw.STL" />
+          <mesh
+            filename="package://so_arm100_description/meshes/Fixed_Jaw.STL"
+          />
+        </geometry>
+        <material name="">
+          <color
+            rgba="0.792156862745098 0.819607843137255 0.933333333333333 1"
+          />
+        </material>
+      </visual>
+      <collision>
+        <origin xyz="0 0 0" rpy="0 0 0" />
+        <geometry>
+          <mesh
+            filename="package://so_arm100_description/meshes/Fixed_Jaw.STL"
+          />
         </geometry>
       </collision>
@@ -282,5 +306,7 @@
         </geometry>
         <material name="">
-          <color rgba="0.792156862745098 0.819607843137255 0.933333333333333 1" />
+          <color
+            rgba="0.792156862745098 0.819607843137255 0.933333333333333 1"
+          />
         </material>
       </visual>
