Commit message: Update SO-100 submodule

File: so_arm100_description/control/so_arm100.ros2_control.xacro (robot description, xacro)
@@ -37,5 +37,5 @@
         <state_interface name="velocity" />
       </joint>
-      <joint name="${prefix}elbow_joint">
+      <joint name="${prefix}elbow_flex_joint">
         <param name="id">3</param>
         <param name="offset">2080</param>
@@ -46,5 +46,5 @@
         <state_interface name="velocity" />
       </joint>
-      <joint name="${prefix}wrist_pitch_joint">
+      <joint name="${prefix}wrist_flex_joint">
         <param name="id">4</param>
         <param name="offset">3110</param>
@@ -64,5 +64,5 @@
         <state_interface name="velocity" />
       </joint>
-      <joint name="${prefix}jaw_joint">
+      <joint name="${prefix}gripper_joint">
         <param name="id">6</param>
         <param name="offset">2070</param>

File: so_arm100_description/urdf/so_arm100.urdf.xacro (robot description, xacro)
@@ -12,7 +12,8 @@
   <xacro:arg name="usb_port" default="/dev/LeRobotFollower" />
   <xacro:arg name="prefix" default="" />
+  <xacro:arg name="color" default="1.0 0.82 0.12 1.0" />
   <!-- Robot description -->
   <xacro:include filename="$(arg urdf_file)" />
-  <xacro:so_arm100 prefix="$(arg prefix)" />
+  <xacro:so_arm100 prefix="$(arg prefix)" color="$(arg color)" />
   <!-- ros2_control description -->
   <xacro:include filename="$(arg ros2_control_file)" />

File: so_arm100_description/urdf/so_arm100_macro.xacro (robot description, xacro)
@@ -1,330 +1,389 @@
 <?xml version="1.0" encoding="utf-8" ?>
 <!-- Copied from
-SO-ARM100/URDF/SO_5DOF_ARM100_8j_URDF.SLDASM/urdf/SO_5DOF_ARM100_8j_URDF.SLDASM.urdf with minimal
-changes:
-- package://SO_5DOF_ARM100_8j_URDF.SLDASM -> package://so_arm100_description
-- Moving Jaw.STL -> Moving_Jaw.STL
-- Link names:
-  - Base -> base
-  - Rotation_Pitch -> shoulder_link
-  - Upper_Arm -> upper_arm_link
-  - Lower_Arm -> forearm_link
-  - Wrist_Pitch_Roll -> wrist_1_link
-  - Fixed_Jaw -> wrist_2_link
-  - Moving Jaw -> jaw_link
-- Joint names:
-  - Rotation -> shoulder_pan_joint
-  - Pitch -> shoulder_lift_joint
-  - Elbow -> elbow_joint
-  - Wrist_Pitch -> wrist_pitch_joint
-  - Wrist_Roll -> wrist_roll_joint
-  - Jaw -> jaw_joint
+SO-ARM100/Simulation/SO100/so100.urdf with minimal changes:
+- Meshes changed to package://so_arm100_description
+- Added parameters for prefix and material color
+- Added _link to link names and _joint to joint names
+- Update default positions and limits of some joints
 -->
 <robot xmlns:xacro="http://ros.org/wiki/xacro">
-  <xacro:macro name="so_arm100" params="prefix">
-    <link name="${prefix}base">
-      <inertial>
-        <origin
-          xyz="-2.45960666746703E-07 0.0311418169687909 0.0175746661003382"
-          rpy="0 0 0"
-        />
-        <mass value="0.193184127927598" />
-        <inertia
-          ixx="0.000137030709467877"
-          ixy="2.10136126944992E-08"
-          ixz="4.24087422551286E-09"
-          iyy="0.000169089551209259"
-          iyz="2.26514711036514E-05"
-          izz="0.000145097720857224"
-        />
-      </inertial>
-      <visual>
+  <xacro:macro name="so_arm100" params="prefix color:='1.0 0.82 0.12 1.0'">
+    <!-- Materials -->
+    <material name="3d_printed">
+      <color rgba="${color}" />
+    </material>
+    <material name="sts3215">
+      <color rgba="0.1 0.1 0.1 1.0" />
+    </material>
+    <!-- Link base -->
+    <link name="${prefix}base_link">
+      <inertial>
+        <!-- Approximate inertial values -->
+        <mass value="1.0" />
         <origin xyz="0 0 0" rpy="0 0 0" />
-        <geometry>
-          <mesh filename="package://so_arm100_description/meshes/Base.STL" />
-        </geometry>
-        <material name="">
-          <color
-            rgba="0.792156862745098 0.819607843137255 0.933333333333333 1"
-          />
-        </material>
-      </visual>
-      <collision>
-        <origin xyz="0 0 0" rpy="0 0 0" />
-        <geometry>
-          <mesh filename="package://so_arm100_description/meshes/Base.STL" />
-        </geometry>
-      </collision>
-    </link>
+        <inertia ixx="0.01" ixy="0" ixz="0" iyy="0.01" iyz="0" izz="0.01" />
+      </inertial>
+      <visual>
+        <geometry>
+          <mesh
+            filename="package://so_arm100_description/SO100/assets/Base.stl"
+          />
+        </geometry>
+        <material name="3d_printed" />
+      </visual>
+      <visual>
+        <geometry>
+          <mesh
+            filename="package://so_arm100_description/SO100/assets/Base_Motor.stl"
+          />
+        </geometry>
+        <material name="sts3215" />
+      </visual>
+      <collision>
+        <geometry>
+          <mesh
+            filename="package://so_arm100_description/SO100/assets/Base.stl"
+          />
+        </geometry>
+      </collision>
+    </link>
+    <!-- Link shoulder -->
     <link name="${prefix}shoulder_link">
       <inertial>
-        <origin
-          xyz="-9.07886224712597E-05 0.0590971820568318 0.031089016892169"
-          rpy="0 0 0"
-        />
-        <mass value="0.119226314127197" />
-        <inertia
-          ixx="5.90408775624429E-05"
-          ixy="4.90800532852998E-07"
-          ixz="-5.90451772654387E-08"
-          iyy="3.21498601038881E-05"
-          iyz="-4.58026206663885E-06"
-          izz="5.86058514263952E-05"
-        />
-      </inertial>
-      <visual>
-        <origin xyz="0 0 0" rpy="0 0 0" />
-        <geometry>
-          <mesh
-            filename="package://so_arm100_description/meshes/Rotation_Pitch.STL"
-          />
-        </geometry>
-        <material name="">
-          <color
-            rgba="0.792156862745098 0.819607843137255 0.933333333333333 1"
-          />
-        </material>
-      </visual>
-      <collision>
-        <origin xyz="0 0 0" rpy="0 0 0" />
-        <geometry>
-          <mesh
-            filename="package://so_arm100_description/meshes/Rotation_Pitch.STL"
-          />
-        </geometry>
-      </collision>
-    </link>
+        <mass value="0.119226" />
+        <origin xyz="-9.07886e-05 0.0590972 0.031089" rpy="0 0 0" />
+        <inertia
+          ixx="5.94278e-05"
+          ixy="0"
+          ixz="0"
+          iyy="5.89975e-05"
+          iyz="0"
+          izz="3.13712e-05"
+        />
+      </inertial>
+      <visual>
+        <geometry>
+          <mesh
+            filename="package://so_arm100_description/SO100/assets/Rotation_Pitch.stl"
+          />
+        </geometry>
+        <material name="3d_printed" />
+      </visual>
+      <visual>
+        <geometry>
+          <mesh
+            filename="package://so_arm100_description/SO100/assets/Rotation_Pitch_Motor.stl"
+          />
+        </geometry>
+        <material name="sts3215" />
+      </visual>
+      <collision>
+        <geometry>
+          <mesh
+            filename="package://so_arm100_description/SO100/assets/Rotation_Pitch.stl"
+          />
+        </geometry>
+      </collision>
+    </link>
+    <!-- Link upper_arm -->
+    <link name="${prefix}upper_arm_link">
+      <inertial>
+        <mass value="0.162409" />
+        <origin xyz="-1.72052e-05 0.0701802 0.00310545" rpy="0 0 0" />
+        <inertia
+          ixx="0.000213312"
+          ixy="0"
+          ixz="0"
+          iyy="0.000167164"
+          iyz="0"
+          izz="7.01522e-05"
+        />
+      </inertial>
+      <visual>
+        <geometry>
+          <mesh
+            filename="package://so_arm100_description/SO100/assets/Upper_Arm.stl"
+          />
+        </geometry>
+        <material name="3d_printed" />
+      </visual>
+      <visual>
+        <geometry>
+          <mesh
+            filename="package://so_arm100_description/SO100/assets/Upper_Arm_Motor.stl"
+          />
+        </geometry>
+        <material name="sts3215" />
+      </visual>
+      <collision>
+        <geometry>
+          <mesh
+            filename="package://so_arm100_description/SO100/assets/Upper_Arm.stl"
+          />
+        </geometry>
+      </collision>
+    </link>
+    <!-- Link lower_arm -->
+    <link name="${prefix}lower_arm_link">
+      <inertial>
+        <mass value="0.147968" />
+        <origin xyz="-0.00339604 0.00137796 0.0768007" rpy="0 0 0" />
+        <inertia
+          ixx="0.000138803"
+          ixy="0"
+          ixz="0"
+          iyy="0.000107748"
+          iyz="0"
+          izz="4.84242e-05"
+        />
+      </inertial>
+      <visual>
+        <geometry>
+          <mesh
+            filename="package://so_arm100_description/SO100/assets/Lower_Arm.stl"
+          />
+        </geometry>
+        <material name="3d_printed" />
+      </visual>
+      <visual>
+        <geometry>
+          <mesh
+            filename="package://so_arm100_description/SO100/assets/Lower_Arm_Motor.stl"
+          />
+        </geometry>
+        <material name="sts3215" />
+      </visual>
+      <collision>
+        <geometry>
+          <mesh
+            filename="package://so_arm100_description/SO100/assets/Lower_Arm.stl"
+          />
+        </geometry>
+      </collision>
+    </link>
+    <!-- Link wrist -->
+    <link name="${prefix}wrist_link">
+      <inertial>
+        <mass value="0.0661321" />
+        <origin xyz="-0.00852653 -0.0352279 -2.34622e-05" rpy="0 0 0" />
+        <inertia
+          ixx="3.45403e-05"
+          ixy="0"
+          ixz="0"
+          iyy="2.39041e-05"
+          iyz="0"
+          izz="1.94704e-05"
+        />
+      </inertial>
+      <visual>
+        <geometry>
+          <mesh
+            filename="package://so_arm100_description/SO100/assets/Wrist_Pitch_Roll.stl"
+          />
+        </geometry>
+        <material name="3d_printed" />
+      </visual>
+      <visual>
+        <geometry>
+          <mesh
+            filename="package://so_arm100_description/SO100/assets/Wrist_Pitch_Roll_Motor.stl"
+          />
+        </geometry>
+        <material name="sts3215" />
+      </visual>
+      <collision>
+        <geometry>
+          <mesh
+            filename="package://so_arm100_description/SO100/assets/Wrist_Pitch_Roll.stl"
+          />
+        </geometry>
+      </collision>
+    </link>
+    <!-- Link gripper -->
+    <link name="${prefix}gripper_link">
+      <inertial>
+        <mass value="0.0929859" />
+        <origin xyz="0.00552377 -0.0280167 0.000483583" rpy="0 0 0" />
+        <inertia
+          ixx="5.03136e-05"
+          ixy="0"
+          ixz="0"
+          iyy="4.64098e-05"
+          iyz="0"
+          izz="2.72961e-05"
+        />
+      </inertial>
+      <visual>
+        <geometry>
+          <mesh
+            filename="package://so_arm100_description/SO100/assets/Fixed_Jaw.stl"
+          />
+        </geometry>
+        <material name="3d_printed" />
+      </visual>
+      <visual>
+        <geometry>
+          <mesh
+            filename="package://so_arm100_description/SO100/assets/Fixed_Jaw_Motor.stl"
+          />
+        </geometry>
+        <material name="sts3215" />
+      </visual>
+    </link>
+    <!-- Link jaw -->
+    <link name="${prefix}jaw_link">
+      <inertial>
+        <mass value="0.0202444" />
+        <origin xyz="-0.00161745 -0.0303473 0.000449646" rpy="0 0 0" />
+        <inertia
+          ixx="1.11265e-05"
+          ixy="0"
+          ixz="0"
+          iyy="8.99651e-06"
+          iyz="0"
+          izz="2.99548e-06"
+        />
+      </inertial>
+      <visual>
+        <geometry>
+          <mesh
+            filename="package://so_arm100_description/SO100/assets/Moving_Jaw.stl"
+          />
+        </geometry>
+        <material name="3d_printed" />
+      </visual>
+    </link>
+    <!-- Joint from base to shoulder -->
     <joint name="${prefix}shoulder_pan_joint" type="revolute">
-      <origin xyz="0 -0.0452 0.0165" rpy="1.5708 0 0" />
-      <parent link="${prefix}base" />
+      <parent link="${prefix}base_link" />
       <child link="${prefix}shoulder_link" />
-      <axis xyz="0 -1 0" />
-      <limit lower="-2.0" upper="2.0" effort="1" velocity="1" />
-    </joint>
-    <link name="${prefix}upper_arm_link">
-      <inertial>
-        <origin
-          xyz="-1.7205170190925E-05 0.0701802156327694 0.00310545118155671"
-          rpy="0 0 0"
-        />
-        <mass value="0.162409284599177" />
-        <inertia
-          ixx="0.000167153146617081"
-          ixy="1.03902689187701E-06"
-          ixz="-1.20161820645189E-08"
-          iyy="7.01946992214245E-05"
-          iyz="2.11884806298698E-06"
-          izz="0.000213280241160769"
-        />
-      </inertial>
-      <visual>
-        <origin xyz="0 0 0" rpy="0 0 0" />
-        <geometry>
-          <mesh
-            filename="package://so_arm100_description/meshes/Upper_Arm.STL"
-          />
-        </geometry>
-        <material name="">
-          <color
-            rgba="0.792156862745098 0.819607843137255 0.933333333333333 1"
-          />
-        </material>
-      </visual>
-      <collision>
-        <origin xyz="0 0 0" rpy="0 0 0" />
-        <geometry>
-          <mesh
-            filename="package://so_arm100_description/meshes/Upper_Arm.STL"
-          />
-        </geometry>
-      </collision>
-    </link>
+      <origin xyz="0 -0.0452 0.0165" rpy="1.57079 0 0" />
+      <axis xyz="0 1 0" />
+      <limit lower="-2" upper="2" effort="35" velocity="1" />
+    </joint>
+    <transmission name="${prefix}shoulder_pan_trans">
+      <type>transmission_interface/SimpleTransmission</type>
+      <joint name="${prefix}shoulder_pan_joint">
+        <hardwareInterface>
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